File: Hardware/Pro/AnySensePro.brd (EAGLE design)
At the start: 26 x 40 mm, 45 parts, among them U1 LP2992IM5-3.3, U3 SN65HVD232D, U4 STM32F303RET6, U6 M25P16VMN6P, X6 MEM2051-00-195-00-A, X7 TC2030-IDC-NL, Y1 ABM3B

Commit message: Final HW Design
Routing:
- net LED_ACTIVITY: track 17.0 -> 10.6 mm
- net LED_ERROR: track 18.8 -> 12.9 mm
- net CANRX: track 25.4 -> 21.1 mm
- net CANTX: track 21.3 -> 17.2 mm
Changed lines of the file:
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@@
 <wire x1="17.355" y1="13.427" x2="17.355" y2="14.688" width="0.1524" layer="1"/>
 <wire x1="17.355" y1="14.688" x2="17.4625" y2="14.7955" width="0.1524" layer="1"/>
-<wire x1="13.589" y1="19.3675" x2="13.589" y2="21.844" width="0.1524" layer="16"/>
-<wire x1="13.589" y1="21.844" x2="14.351" y2="22.606" width="0.1524" layer="16"/>
-<wire x1="14.351" y1="22.606" x2="16.891" y2="22.606" width="0.1524" layer="16"/>
-<wire x1="16.891" y1="22.606" x2="17.399" y2="23.114" width="0.1524" layer="16"/>
+<wire x1="16.764" y1="22.479" x2="17.399" y2="23.114" width="0.1524" layer="16"/>
 <wire x1="17.399" y1="23.114" x2="17.399" y2="24.003" width="0.1524" layer="16"/>
-<wire x1="13.589" y1="19.3675" x2="17.4625" y2="15.494" width="0.15" layer="16"/>
-<wire x1="17.4625" y1="15.494" x2="17.4625" y2="14.7955" width="0.15" layer="16"/>
+<wire x1="16.764" y1="22.479" x2="16.764" y2="20.955" width="0.1524" layer="16"/>
+<wire x1="16.764" y1="20.955" x2="17.4625" y2="20.2565" width="0.1524" layer="16"/>
+<wire x1="17.4625" y1="20.2565" x2="17.4625" y2="14.7955" width="0.1524" layer="16"/>
 </signal>
 <signal name="CANRX">
@@
 <wire x1="16.764" y1="15.367" x2="16.855" y2="15.276" width="0.1524" layer="1"/>
 <wire x1="16.855" y1="15.276" x2="16.855" y2="13.427" width="0.1524" layer="1"/>
-<wire x1="16.764" y1="15.367" x2="13.081" y2="19.05" width="0.1524" layer="16"/>
-<wire x1="13.081" y1="19.05" x2="13.081" y2="22.098" width="0.1524" layer="16"/>
-<wire x1="13.081" y1="22.098" x2="13.97" y2="22.987" width="0.1524" layer="16"/>
-<wire x1="13.97" y1="22.987" x2="16.764" y2="22.987" width="0.1524" layer="16"/>
-<wire x1="16.764" y1="22.987" x2="17.018" y2="23.241" width="0.1524" layer="16"/>
 <wire x1="17.018" y1="23.241" x2="17.018" y2="23.876" width="0.1524" layer="16"/>
+<wire x1="17.018" y1="23.241" x2="16.383" y2="22.606" width="0.1524" layer="16"/>
+<wire x1="16.383" y1="22.606" x2="16.383" y2="20.828" width="0.1524" layer="16"/>
+<wire x1="16.383" y1="20.828" x2="16.891" y2="20.32" width="0.1524" layer="16"/>
+<wire x1="16.891" y1="20.32" x2="16.891" y2="15.494" width="0.1524" layer="16"/>
+<wire x1="16.891" y1="15.494" x2="16.764" y2="15.367" width="0.1524" layer="16"/>
 </signal>
 <signal name="SWDIO">
@@
 <wire x1="9.906" y1="11.938" x2="7.239" y2="11.938" width="0.1524" layer="16"/>
 <wire x1="7.239" y1="11.938" x2="5.588" y2="10.287" width="0.1524" layer="16"/>
+<via x="6.985" y="8.128" extent="1-16" drill="0.25"/>
+<wire x1="6.985" y1="8.128" x2="7.747" y2="8.89" width="0.15" layer="1"/>
 <wire x1="5.588" y1="10.287" x2="5.588" y2="9.144" width="0.1524" layer="16"/>
 <wire x1="5.588" y1="9.144" x2="6.604" y2="8.128" width="0.1524" layer="16"/>
 <wire x1="6.604" y1="8.128" x2="6.985" y2="8.128" width="0.1524" layer="16"/>
-<via x="6.985" y="8.128" extent="1-16" drill="0.25"/>
-<wire x1="6.985" y1="8.128" x2="7.747" y2="8.89" width="0.15" layer="1"/>
 </signal>
 <signal name="SWCLK">
@@
 <wire x1="10.474" y1="12.446" x2="10.855" y2="12.827" width="0.1524" layer="1"/>
 <via x="5.715" y="8.128" extent="1-16" drill="0.25"/>
-<wire x1="5.715" y1="8.128" x2="5.588" y2="8.128" width="0.1524" layer="16"/>
-<wire x1="5.588" y1="8.128" x2="5.207" y2="8.636" width="0.1524" layer="16"/>
-<wire x1="5.207" y1="8.636" x2="5.207" y2="10.541" width="0.1524" layer="16"/>
 <wire x1="5.207" y1="10.541" x2="7.112" y2="12.446" width="0.1524" layer="16"/>
 <wire x1="7.112" y1="12.446" x2="9.5885" y2="12.446" width="0.1524" layer="16"/>
@@
 <wire x1="6.096" y1="8.128" x2="6.477" y2="8.509" width="0.15" layer="1"/>
 <wire x1="6.477" y1="8.509" x2="6.477" y2="8.89" width="0.15" layer="1"/>
+<wire x1="5.207" y1="10.541" x2="5.207" y2="8.509" width="0.1524" layer="16"/>
+<wire x1="5.207" y1="8.509" x2="5.588" y2="8.128" width="0.1524" layer="16"/>
+<wire x1="5.588" y1="8.128" x2="5.715" y2="8.128" width="0.1524" layer="16"/>
 </signal>
 <signal name="TRACESWO">
@@
 <via x="13.081" y="23.622" extent="1-16" drill="0.25"/>
 <via x="14.351" y="19.431" extent="1-16" drill="0.25"/>
-<via x="16.002" y="17.78" extent="1-16" drill="0.25"/>
-<via x="17.78" y="17.78" extent="1-16" drill="0.25"/>
+<via x="16.256" y="17.78" extent="1-16" drill="0.25"/>
+<via x="18.161" y="17.78" extent="1-16" drill="0.25"/>
 <via x="17.526" y="35.433" extent="1-16" drill="0.25"/>
-<via x="16.002" y="19.3675" extent="1-16" drill="0.25"/>
-<via x="17.78" y="19.3675" extent="1-16" drill="0.25"/>
+<via x="16.256" y="19.431" extent="1-16" drill="0.25"/>
+<via x="18.161" y="19.4945" extent="1-16" drill="0.25"/>
 <via x="12.319" y="20.32" extent="1-16" drill="0.25"/>
 <via x="12.319" y="19.431" extent="1-16" drill="0.25"/>
 <via x="12.319" y="21.717" extent="1-16" drill="0.25"/>
-<via x="11.303" y="22.733" extent="1-16" drill="0.25"/>
+<via x="11.049" y="23.622" extent="1-16" drill="0.25"/>
 <via x="10.287" y="22.733" extent="1-16" drill="0.25"/>
 <via x="10.287" y="21.717" extent="1-16" drill="0.25"/>
@@
 <via x="6.787" y="22.933" extent="1-16" drill="0.25"/>
 <via x="7.887" y="24.033" extent="1-16" drill="0.25"/>
-<via x="4.287" y="25.333" extent="1-16" drill="0.25"/>
+<via x="3.779" y="25.714" extent="1-16" drill="0.25"/>
 <via x="3.787" y="29.433" extent="1-16" drill="0.25"/>
 <via x="8.187" y="25.433" extent="1-16" drill="0.25"/>
@@
 <via x="9.398" y="14.097" extent="1-16" drill="0.25"/>
 <via x="10.033" y="15.875" extent="1-16" drill="0.25"/>
-<via x="17.78" y="16.002" extent="1-16" drill="0.25"/>
+<via x="18.161" y="16.383" extent="1-16" drill="0.25"/>
 <via x="14.351" y="8.89" extent="1-16" drill="0.25"/>
 <via x="19.177" y="17.78" extent="1-16" drill="0.25"/>
@@
 <via x="23.876" y="33.401" extent="1-16" drill="0.25"/>
 <via x="19.05" y="27.305" extent="1-16" drill="0.25"/>
+<via x="14.351" y="20.32" extent="1-16" drill="0.25"/>
+<via x="16.002" y="20.32" extent="1-16" drill="0.25"/>
+<via x="24.003" y="21.463" extent="1-16" drill="0.25"/>
+<via x="24.003" y="19.431" extent="1-16" drill="0.25"/>
+<via x="24.003" y="17.653" extent="1-16" drill="0.25"/>
+<via x="21.59" y="18.669" extent="1-16" drill="0.25"/>
+<via x="4.287" y="24.444" extent="1-16" drill="0.25"/>
+<via x="14.351" y="17.78" extent="1-16" drill="0.25"/>
+<via x="16.002" y="16.002" extent="1-16" drill="0.25"/>
+<via x="14.351" y="22.225" extent="1-16" drill="0.25"/>
 </signal>
 <signal name="CANL">
@@
 <via x="19.812" y="26.7335" extent="1-16" drill="0.25"/>
 <wire x1="17.907" y1="25.273" x2="17.907" y2="22.987" width="0.1524" layer="16"/>
-<wire x1="17.907" y1="22.987" x2="17.145" y2="22.225" width="0.1524" layer="16"/>
-<wire x1="17.145" y1="22.225" x2="14.605" y2="22.225" width="0.1524" layer="16"/>
-<wire x1="14.605" y1="22.225" x2="14.097" y2="21.717" width="0.1524" layer="16"/>
-<wire x1="14.097" y1="21.717" x2="14.097" y2="20.574" width="0.1524" layer="16"/>
-<wire x1="14.097" y1="20.574" x2="14.732" y2="19.939" width="0.1524" layer="16"/>
-<wire x1="14.732" y1="19.939" x2="18.923" y2="19.939" width="0.1524" layer="16"/>
 <wire x1="18.923" y1="19.939" x2="19.177" y2="19.685" width="0.1524" layer="16"/>
 <via x="19.177" y="19.685" extent="1-16" drill="0.25"/>
@@
 <wire x1="17.907" y1="25.273" x2="19.3675" y2="26.7335" width="0.1524" layer="16"/>
 <wire x1="19.3675" y1="26.7335" x2="19.812" y2="26.7335" width="0.1524" layer="16"/>
+<wire x1="17.907" y1="22.987" x2="17.272" y2="22.352" width="0.1524" layer="16"/>
+<wire x1="17.272" y1="22.352" x2="17.272" y2="20.955" width="0.1524" layer="16"/>
+<wire x1="17.272" y1="20.955" x2="18.034" y2="20.193" width="0.1524" layer="16"/>
+<wire x1="18.034" y1="20.193" x2="18.669" y2="20.193" width="0.1524" layer="16"/>
+<wire x1="18.669" y1="20.193" x2="19.177" y2="19.685" width="0.1524" layer="16"/>
 </signal>
 <signal name="LED_ACTIVITY">
@@
 <wire x1="19.05" y1="25.908" x2="18.288" y2="25.146" width="0.1524" layer="16"/>
 <wire x1="18.288" y1="25.146" x2="18.288" y2="22.86" width="0.1524" layer="16"/>
-<wire x1="18.288" y1="22.86" x2="17.272" y2="21.844" width="0.1524" layer="16"/>
-<wire x1="17.272" y1="21.844" x2="14.732" y2="21.844" width="0.1524" layer="16"/>
-<wire x1="14.732" y1="21.844" x2="14.478" y2="21.59" width="0.1524" layer="16"/>
-<wire x1="14.478" y1="21.59" x2="14.478" y2="20.701" width="0.1524" layer="16"/>
-<wire x1="14.478" y1="20.701" x2="14.859" y2="20.32" width="0.1524" layer="16"/>
-<wire x1="14.859" y1="20.32" x2="18.923" y2="20.32" width="0.1524" layer="16"/>
-<wire x1="18.923" y1="20.32" x2="19.177" y2="20.574" width="0.1524" layer="16"/>
 <via x="19.177" y="20.574" extent="1-16" drill="0.25"/>
 <wire x1="19.177" y1="20.574" x2="19.324" y2="20.427" width="0.1524" layer="1"/>
@@
 <wire x1="21.275" y1="25.989" x2="19.893" y2="25.989" width="0.1524" layer="1"/>
 <wire x1="19.893" y1="25.989" x2="19.812" y2="25.908" width="0.1524" layer="1"/>
+<wire x1="18.288" y1="22.86" x2="17.653" y2="22.225" width="0.1524" layer="16"/>
+<wire x1="17.653" y1="22.225" x2="17.653" y2="21.082" width="0.1524" layer="16"/>
+<wire x1="17.653" y1="21.082" x2="18.161" y2="20.574" width="0.1524" layer="16"/>
+<wire x1="18.161" y1="20.574" x2="19.177" y2="20.574" width="0.1524" layer="16"/>
 </signal>
 <signal name="N$15">
